Commit message: gazebo

File: src/mastering_ros_robot_description_pkg/urdf/diff_wheeled_robot_with_laser.xacro (robot description, xacro)
@@ -42,4 +42,48 @@
   <!-- Hokuyo Laser scanner -->
   <xacro:property name="hokuyo_size" value="0.05" />
+  <xacro:property name="laser_height" value="0.08" />
+  <!-- 기둥관련 : 기둥 위치: base_radius -0.02, 기둥높이: 0.08m 기둥반지름: 0.005m -->
+  <xacro:property name="pillar_radius" value="0.005" />
+  <xacro:property name="pillar_height" value="0.08" />
+  <xacro:property name="pillar_offset" value="0.10" />
+  <xacro:property name="pillar_mass" value="0.1" />
+  <!-- 기둥의 메크로 정의  -->
+  <xacro:macro name="pillar" params="name x y">
+  <link name="${name}">
+  <visual>
+  <origin xyz="0 0 ${pillar_height/2}" rpy="0 0 0"/>
+  <geometry>
+  <cylinder length="${pillar_height}" radius="${pillar_radius}"  />
+  </geometry>
+  <material name="Black"/>
+  </visual>
+  <collision>
+  <origin xyz- "0 0 ${pillar_height/2}" radius="0 0 0"/>
+  <geometry>
+  <cylinder length="${pillar_height}" radius="${pillar_radius}"/>
+  </geometry>
+  </collision>
+  <inertial>
+  <mass value="${pillar_masss}"/>
+  <origin xyz="0 0 ${pillar_height/2}"/>
+  <inertia ixx="0.001" ixy="0.0" ixz="0.0"
+           iyy="0.0001" iyz="0.0"
+           izz="0.0001"/>
+  </inertia>
+  </link>
+  <join name="${name}_joint" type="fixed">
+  <parent link="Sbase_link"/>
+  <child link="${name}"/>
+  <origin xyz="${x} ${y} ${base_height/2}" rpy="0 0 0"/>
+  </joint>
+  <gazebo reference="${name}"/>
+  <material>Gazebo/Black</material>
+  </gazebo>
+</xacro:macro>
+<!-- 기둥 4개 배치(사각형 모서리) -->
+<xacro:pillar name="pillar_front_left" x="${pillar_offset}" y="${pillar_offset}"/>
+<xacro:pillar name="pillar_front_right" x="${pillar_offset}" y="${pillar_offset}"/>
+<xacro:pillar name="pillar_back_left" x="${-pillar_offset}" y="${pillar_offset}"/>
+<xacro:pillar name="pillar_back_right" x="${-pillar_offset}" y="${pillar_offset}"/>
   <!-- Macro for calculating inertia of cylinder -->
   <xacro:macro name="cylinder_inertia" params="m r h">
@@ -195,5 +239,6 @@
   </link>
   <joint name="hokuyo_joint" type="fixed">
-    <origin xyz="${base_radius - hokuyo_size/2} 0 ${base_height+hokuyo_size/4}" rpy="0 0 0" />
+    <!-- <origin xyz="${base_radius - hakuyo_size/2} 0 ${base_height+hokuyo_size/4}" rpy="0 0 0" /> -->
+    <origin xyz=" 0 0 ${base_height+hokuyo_size/4}" rpy="0 0 0" />
     <parent link="base_link"/>
     <child link="laser_link" />
@@ -211,6 +256,6 @@
             <samples>720</samples>
             <resolution>1</resolution>
-            <min_angle>-1.570796</min_angle>
-            <max_angle>1.570796</max_angle>
+            <min_angle>-3.14159</min_angle>
+            <max_angle>3.14159</max_angle>
           </horizontal>
         </scan>
